Commit message: ttyPORT changed + modified xacro

File: pantilt_bot_description/urdf/pantilt_bot.ros2_control.xacro (robot description, xacro)
@@ -25,4 +25,12 @@
         <state_interface name="effort"/>
       </joint>
+      <joint name="joint3">
+        <param name="id">13</param>
+        <command_interface name="position"/>
+        <command_interface name="velocity"/>
+        <state_interface name="position"/>
+        <state_interface name="velocity"/>
+        <state_interface name="effort"/>
+      </joint>
     </ros2_control>
   </xacro:macro>

File: pantilt_bot_description/urdf/pantilt_bot.ros2_control_gazebo.xacro (robot description, xacro)
@@ -20,4 +20,11 @@
         <state_interface name="effort"/>
       </joint>
+      <joint name="joint3">
+        <command_interface name="position"/>
+        <command_interface name="velocity"/>
+        <state_interface name="position"/>
+        <state_interface name="velocity"/>
+        <state_interface name="effort"/>
+      </joint>
     </ros2_control>
     <gazebo>

File: pantilt_bot_description/urdf/pantilt_bot.urdf.xacro (robot description, xacro)
@@ -3,12 +3,12 @@
   <xacro:include filename="$(find pantilt_bot_description)/urdf/pantilt_bot.xacro" />
   <xacro:include filename="$(find pantilt_bot_description)/urdf/pantilt_bot.ros2_control.xacro" />
-  <xacro:include filename="$(find realsense2_description)/urdf/_d435.urdf.xacro" />
+  <!--xacro:include filename="$(find realsense2_description)/urdf/_d435.urdf.xacro" /-->
   <link name="world"/>
   <xacro:pantilt_bot parent="world">
     <origin xyz="0 0 0" rpy="0 0 0" />
   </xacro:pantilt_bot>
-  <xacro:sensor_d435 parent="joint2_horn_link" use_nominal_extrinsics="true" add_plug="false">
+  <!--xacro:sensor_d435 parent="joint2_horn_link" use_nominal_extrinsics="true" add_plug="false">
     <origin xyz="-0.0125 -0.019 0.065" rpy="0 -1.5708 3.1416"/>
-  </xacro:sensor_d435>
+  </xacro:sensor_d435-->
   <xacro:pantilt_bot_ros2_control name="pantilt_bot_ros2_control" />
 </robot>

File: pantilt_bot_description/urdf/pantilt_bot.xacro (robot description, xacro)
@@ -4,5 +4,10 @@
   <xacro:include filename="$(find pantilt_bot_description)/urdf/pantilt_bot.material.xacro" />
   <xacro:macro name="pantilt_bot" params="parent *origin">
-    <link name="joint1_link">
+    <joint name="origin_to_link_0" type="fixed">
+      <xacro:insert_block name="origin" />
+      <parent link="${parent}" />
+      <child link="link_0" />
+    </joint>
+    <link name="link_0">
       <inertial>
         <origin rpy="0 0 0" xyz="-5.549338143508866e-15 0.011937164947263951 0.019605935309866387"/>
@@ -13,5 +18,5 @@
         <origin rpy="0 0 0" xyz="0 0 0"/>
         <geometry>
-          <mesh filename="package://pantilt_bot_description/meshes/joint1.stl" scale="0.001 0.001 0.001"/>
+          <mesh filename="package://pantilt_bot_description/meshes/link_0.stl" scale="0.001 0.001 0.001"/>
         </geometry>
         <material name="grey"/>
@@ -20,9 +25,16 @@
         <origin rpy="0 0 0" xyz="0 0 0"/>
         <geometry>
-          <mesh filename="package://pantilt_bot_description/meshes/joint1.stl" scale="0.001 0.001 0.001"/>
+          <mesh filename="package://pantilt_bot_description/meshes/link_0.stl" scale="0.001 0.001 0.001"/>
         </geometry>
       </collision>
     </link>
-    <link name="joint1_horn_link">
+    <joint name="joint1" type="revolute">
+      <origin rpy="0 0 1.5708" xyz="0.0 0.000319 0.038"/>
+      <parent link="link_0"/>
+      <child link="link_1_horn"/>
+      <axis xyz="-0.0 -0.0 1.0"/>
+      <limit effort="1" lower="-2.96706" upper="2.96706" velocity="${46 / 60.0 * 2.0 * pi}"/>
+    </joint>
+    <link name="link_1_horn">
       <inertial>
         <origin rpy="0 0 0" xyz="7.323601717155284e-17 -3.584248942771506e-07 0.0027880990797749597"/>
@@ -33,5 +45,5 @@
         <origin rpy="0 0 0" xyz="0.0 -0.000319 -0.038"/>
         <geometry>
-          <mesh filename="package://pantilt_bot_description/meshes/joint1_horn.stl" scale="0.001 0.001 0.001"/>
+          <mesh filename="package://pantilt_bot_description/meshes/link_1_horn.stl" scale="0.001 0.001 0.001"/>
         </geometry>
         <material name="grey"/>
@@ -40,9 +52,14 @@
         <origin rpy="0 0 0" xyz="0.0 -0.000319 -0.038"/>
         <geometry>
-          <mesh filename="package://pantilt_bot_description/meshes/joint1_horn.stl" scale="0.001 0.001 0.001"/>
+          <mesh filename="package://pantilt_bot_description/meshes/link_1_horn.stl" scale="0.001 0.001 0.001"/>
         </geometry>
       </collision>
     </link>
-    <link name="joint2_link">
+    <joint name="joint_link1_horn2motor" type="fixed">
+      <origin rpy="0 0 0" xyz="0.011 -0.017 0.0085"/>
+      <parent link="link_1_horn"/>
+      <child link="link_1_motor"/>
+    </joint>
+    <link name="link_1_motor">
       <inertial>
         <origin rpy="0 0 0" xyz="-0.010999999999994571 0.016393706265213467 0.02038147662781581"/>
@@ -53,5 +70,5 @@
         <origin rpy="0 0 0" xyz="-0.011 0.016681 -0.0465"/>
         <geometry>
-          <mesh filename="package://pantilt_bot_description/meshes/joint2.stl" scale="0.001 0.001 0.001"/>
+          <mesh filename="package://pantilt_bot_description/meshes/link_1_motor.stl" scale="0.001 0.001 0.001"/>
         </geometry>
         <material name="grey"/>
@@ -60,51 +77,86 @@
         <origin rpy="0 0 0" xyz="-0.011 0.016681 -0.0465"/>
         <geometry>
-          <mesh filename="package://pantilt_bot_description/meshes/joint2.stl" scale="0.001 0.001 0.001"/>
+          <mesh filename="package://pantilt_bot_description/meshes/link_1_motor.stl" scale="0.001 0.001 0.001"/>
         </geometry>
       </collision>
     </link>
-    <link name="joint2_horn_link">
+    <joint name="joint2" type="revolute">
+      <origin rpy="0 0 0" xyz="-0.011 0.036 0.032"/>
+      <parent link="link_1_motor"/>
+      <child link="link_2"/>
+      <axis xyz="-0.0 -1.0 -0.0"/>
+      <limit effort="1" lower="-2.1" upper="2.1" velocity="${46 / 60.0 * 2.0 * pi}"/>
+    </joint>
+    <link name="link_2">
       <inertial>
         <origin rpy="0 0 0" xyz="7.674625448279525e-16 -0.019000358424909176 0.03767262835995369"/>
-        <mass value="0.05331898839844395"/>
+        <mass value="0.105331898839844395"/>
         <inertia ixx="3.2e-05" ixy="-0.0" ixz="0.0" iyy="2e-05" iyz="-0.0" izz="1.9e-05"/>
       </inertial>
       <visual>
-        <origin rpy="0 0 0" xyz="-0.0 -0.019319 -0.0785"/>
+        <origin rpy="0 -1.57 0" xyz="0.02 -0.05 -0.02"/>
         <geometry>
-          <mesh filename="package://pantilt_bot_description/meshes/joint2_horn.stl" scale="0.001 0.001 0.001"/>
+          <mesh filename="package://pantilt_bot_description/meshes/link_2.stl" scale="0.01 0.01 0.01"/>
         </geometry>
         <material name="grey"/>
       </visual>
       <collision>
-        <origin rpy="0 0 0" xyz="-0.0 -0.019319 -0.0785"/>
+        <origin rpy="0 -1.57 0" xyz="0.02 -0.05 -0.02"/>
         <geometry>
-          <mesh filename="package://pantilt_bot_description/meshes/joint2_horn.stl" scale="0.001 0.001 0.001"/>
+          <mesh filename="package://pantilt_bot_description/meshes/link_2.stl" scale="0.01 0.01 0.01"/>
         </geometry>
       </collision>
     </link>
-    <joint name="origin_to_joint1" type="fixed">
-      <xacro:insert_block name="origin" />
-      <parent link="${parent}" />
-      <child link="joint1_link" />
+    <joint name="joint3" type="revolute">
+      <origin rpy="0 0 0" xyz="0 0 0.42"/>
+      <parent link="link_2"/>
+      <child link="link_3_motor"/>
+      <axis xyz="-0.0 1.0 -0.0"/>
+      <limit effort="1" lower="-2.1" upper="2.1" velocity="${46 / 60.0 * 2.0 * pi}"/>
     </joint>
-    <joint name="joint1" type="revolute">
-      <origin rpy="0 0 1.5708" xyz="0.0 0.000319 0.038"/>
-      <parent link="joint1_link"/>
-      <child link="joint1_horn_link"/>
-      <axis xyz="-0.0 -0.0 1.0"/>
-      <limit effort="1" lower="-2.96706" upper="2.96706" velocity="${46 / 60.0 * 2.0 * pi}"/>
-    </joint>
-    <joint name="joint1_horn_to_joint2" type="fixed">
-      <origin rpy="0 0 0" xyz="0.011 -0.017 0.0085"/>
-      <parent link="joint1_horn_link"/>
-      <child link="joint2_link"/>
-    </joint>
-    <joint name="joint2" type="revolute">
-      <origin rpy="0 0 0" xyz="-0.011 0.036 0.032"/>
-      <parent link="joint2_link"/>
-      <child link="joint2_horn_link"/>
-      <axis xyz="-0.0 -1.0 -0.0"/>
-      <limit effort="1" lower="-2.1" upper="2.1" velocity="${46 / 60.0 * 2.0 * pi}"/>
+    <link name="link_3_motor">
+      <inertial>
+        <origin rpy="0 0 0" xyz="-0.010999999999994571 0.016393706265213467 0.02038147662781581" />
+        <mass value="0.34009000706899195"/>
+        <inertia ixx="9.4e-05" ixy="0.0" ixz="-0.0" iyy="8.2e-05" iyz="0.0" izz="5.5e-05"/>
+      </inertial>
+      <visual>
+        <origin rpy="0 3.14 0" xyz="0.0 -0.02 0.078"/>
+        <geometry>
+          <mesh filename="package://pantilt_bot_description/meshes/link_3_motor.stl" scale="0.001 0.001 0.001"/>
+        </geometry>
+        <material name="grey"/>
+      </visual>
+      <collision>
+        <origin rpy="0 3.14 0" xyz="0.0 -0.02 0.078"/>
+        <geometry>
+          <mesh filename="package://pantilt_bot_description/meshes/link_3_motor.stl" scale="0.001 0.001 0.001"/>
+        </geometry>
+      </collision>
+    </link>
+    <link name="link_3_horn">
+      <inertial>
+        <origin rpy="0 0 0" xyz="7.323601717155284e-17 -3.584248942771506e-07 0.0027880990797749597"/>
+        <mass value="0.016309929358964557"/>
+        <inertia ixx="3e-06" ixy="-0.0" ixz="-0.0" iyy="1e-06" iyz="0.0" izz="4e-06"/>
+      </inertial>
+      <visual>
+        <origin rpy="0 1.57 0" xyz="-0.0175 -0.001 0.36"/>
+        <geometry>
+          <mesh filename="package://pantilt_bot_description/meshes/link_3_horn.stl" scale="0.01 0.01 0.01"/>
+        </geometry>
+        <material name="grey"/>
+      </visual>
+      <collision>
+        <origin rpy="0 1.57 0" xyz="0.0 -0.000319 -0.038"/>
+        <geometry>
+          <mesh filename="package://pantilt_bot_description/meshes/link_3_horn.stl" scale="0.01 0.01 0.01"/>
+        </geometry>
+      </collision>
+    </link>
+    <joint name="joint_link3_motor2horn" type="fixed">
+      <origin rpy="0 0 0" xyz="-0 0 0"/>
+      <parent link="link_3_motor"/>
+      <child link="link_3_horn"/>
     </joint>
   </xacro:macro>

File: pantilt_bot_description/urdf/pantilt_bot_gazebo.urdf.xacro (robot description, xacro)
@@ -3,12 +3,12 @@
   <xacro:include filename="$(find pantilt_bot_description)/urdf/pantilt_bot.xacro" />
   <xacro:include filename="$(find pantilt_bot_description)/urdf/pantilt_bot.ros2_control_gazebo.xacro" />
-  <xacro:include filename="$(find realsense2_description)/urdf/_d435.urdf.xacro" />
+  <!--xacro:include filename="$(find realsense2_description)/urdf/_d435.urdf.xacro" /-->
   <link name="world"/>
   <xacro:pantilt_bot parent="world">
     <origin xyz="0 0 0" rpy="0 0 0" />
   </xacro:pantilt_bot>
-  <xacro:sensor_d435 parent="joint2_horn_link" use_nominal_extrinsics="true" add_plug="false">
+  <!--xacro:sensor_d435 parent="joint2_horn_link" use_nominal_extrinsics="true" add_plug="false">
     <origin xyz="-0.0125 -0.019 0.065" rpy="0 -1.5708 3.1416"/>
-  </xacro:sensor_d435>
+  </xacro:sensor_d435-->
   <xacro:pantilt_bot_ros2_control name="pantilt_bot_ros2_control" />
 </robot>
